File: JPBms2.kicad_pcb (KiCad board)
At the start: 4 copper layers, 68.2 x 38.2 mm, 89 parts, among them J1 Conn_ARM_SWD_TagConnect_TC2030, J2 Barrel_Jack_MountingPin, Q1 AO3401A, Q10 AO3401A, Q11 2N7002, Q2 AO3401A, Q3 AO3400A, Q4 AO3400A, Q5 AO3401A, Q6 2N7002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

Commit message: More layout adust
Parts:
- C14, C15: footprint Capacitor_SMD:C_0805_2012Metric -> Capacitor_SMD:C_1206_3216Metric
- moved C19 91.0 mm to (140.5, 75.3), turned to 90 degrees
- moved C18 90.9 mm to (140.5, 72.0), turned to 90 degrees
- moved R27 88.0 mm to (138.2, 71.1)
- moved R29 88.0 mm to (138.2, 76.1)
- moved R28 87.8 mm to (138.2, 72.8), turned to 180 degrees
- moved R30 87.6 mm to (138.2, 74.4), turned to 180 degrees
- moved R7 85.8 mm to (134.7, 82.2), turned to 90 degrees
- moved R8 80.2 mm to (131.8, 82.2), turned to 90 degrees
- moved C12 76.4 mm to (133.3, 82.2), turned to -90 degrees
- moved C3 73.4 mm to (130.3, 82.2), turned to -90 degrees
- moved C4 70.5 mm to (122.8, 80.4), turned to 90 degrees
- moved D8 65.7 mm to (134.9, 74.9), turned to 180 degrees
- moved D7 64.7 mm to (134.9, 72.3), turned to 180 degrees
- moved C15 55.5 mm to (153.9, 86.6), turned to -90 degrees
- moved C14 54.6 mm to (153.8, 77.5), turned to 90 degrees
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Connections:
- C14 pad 1: +BATT -> Net-(U3-Vs+)
- C15 pad 1: VSOLAR -> Net-(U3-Vs+)
Routing:
- net Net-(U5-LO): track 0.00 -> 9.82 mm
- net Net-(U3-Vs-): track 0.00 -> 3.91 mm
- net /BuckBoost/GATE_BOT_B: track 0.00 -> 2.42 mm
- net /BuckBoost/GATE_TOP_B: track 0.00 -> 2.39 mm
- net Net-(U3-Vs+): track 0.00 -> 2.39 mm
- net Net-(D2-K): track 0.00 -> 1.78 mm
- net Net-(D3-K): track 0.00 -> 1.60 mm
- net Net-(D1-K): track 0.00 -> 1.60 mm
Other:
- board text added: "PozSolarChg v1.0"

Commit message: Smallfixups
Parts:
- moved C10 18.4 mm to (132.0, 75.9), turned to -90 degrees
- moved C6 9.76 mm to (116.5, 73.7)
- moved C9 1.44 mm to (118.3, 73.7)
Changed lines of the file:
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@@
 	(footprint "Capacitor_SMD:C_0603_1608Metric"
 		(layer "F.Cu")
-		(at 117.5 64.5 90)
+		(at 131.953 75.946 -90)
 		(descr "Capacitor SMD 0603 (1608 Metric), square (rectangular) end terminal, IPC_7351 nominal, (Body size source: IPC-SM-782 page 76, https://www.pcb-3d.com/wordpress/wp-content/uploads/ipc-sm-782a_amendment_1_and_2.pdf), generated with kicad-footprint-generator")
 		(tags "capacitor")
 		(property "Reference" "C10"
-			(at 0 -1.43 -90)
+			(at 0 -1.43 90)
 			(layer "F.SilkS")
 			(effects
@@
 		)
 		(property "Value" ".1u"
-			(at 0 1.43 -90)
+			(at 0 1.43 90)
 			(layer "F.Fab")
 			(effects
@@
 		)
 		(property "Footprint" "Capacitor_SMD:C_0603_1608Metric"
-			(at 0 0 90)
+			(at 0 0 -90)
 			(unlocked yes)
 			(layer "F.Fab")
@@
 		)
 		(property "Datasheet" ""
-			(at 0 0 90)
+			(at 0 0 -90)
 			(unlocked yes)
 			(layer "F.Fab")
@@
 		)
 		(property "Description" "Unpolarized capacitor, small symbol"
-			(at 0 0 90)
+			(at 0 0 -90)
 			(unlocked yes)
 			(layer "F.Fab")
@@
 		)
 		(property "LCSC_Code" "C14663"
-			(at 0 0 90)
+			(at 0 0 -90)
 			(unlocked yes)
 			(layer "F.Fab")
@@
 		(attr smd)
 		(fp_line
-			(start -0.14058 -0.51)
-			(end 0.14058 -0.51)
+			(start -0.14058 0.51)
+			(end 0.14058 0.51)
 			(stroke
 				(width 0.12)
@@
 		)
 		(fp_line
-			(start -0.14058 0.51)
-			(end 0.14058 0.51)
+			(start -0.14058 -0.51)
+			(end 0.14058 -0.51)
 			(stroke
 				(width 0.12)
@@
 		)
 		(fp_line
-			(start 1.48 -0.73)
-			(end 1.48 0.73)
+			(start -1.48 0.73)
+			(end -1.48 -0.73)
 			(stroke
 				(width 0.05)
@@
 		)
 		(fp_line
-			(start -1.48 -0.73)
-			(end 1.48 -0.73)
+			(start 1.48 0.73)
+			(end -1.48 0.73)
 			(stroke
 				(width 0.05)
@@
 		)
 		(fp_line
-			(start 1.48 0.73)
-			(end -1.48 0.73)
+			(start -1.48 -0.73)
+			(end 1.48 -0.73)
 			(stroke
 				(width 0.05)
@@
 		)
 		(fp_line
-			(start -1.48 0.73)
-			(end -1.48 -0.73)
+			(start 1.48 -0.73)
+			(end 1.48 0.73)
 			(stroke
 				(width 0.05)
@@
 		)
 		(fp_line
-			(start 0.8 -0.4)
-			(end 0.8 0.4)
+			(start -0.8 0.4)
+			(end -0.8 -0.4)
 			(stroke
 				(width 0.1)
@@
 		)
 		(fp_line
-			(start -0.8 -0.4)
-			(end 0.8 -0.4)
+			(start 0.8 0.4)
+			(end -0.8 0.4)
 			(stroke
 				(width 0.1)
@@
 		)
 		(fp_line
-			(start 0.8 0.4)
-			(end -0.8 0.4)
+			(start -0.8 -0.4)
+			(end 0.8 -0.4)
 			(stroke
 				(width 0.1)
@@
 		)
 		(fp_line
-			(start -0.8 0.4)
-			(end -0.8 -0.4)
+			(start 0.8 -0.4)
+			(end 0.8 0.4)
 			(stroke
 				(width 0.1)
@@
 		)
 		(fp_text user "${REFERENCE}"
-			(at 0 0 -90)
+			(at 0 0 90)
 			(layer "F.Fab")
 			(effects
@@
 		)
 		(pad "1" smd roundrect
-			(at -0.775 0 90)
+			(at -0.775 0 270)
 			(size 0.9 0.95)
 			(layers "F.Cu" "F.Paste" "F.Mask")
@@
 		)
 		(pad "2" smd roundrect
-			(at 0.775 0 90)
+			(at 0.775 0 270)
 			(size 0.9 0.95)
 			(layers "F.Cu" "F.Paste" "F.Mask")
@@
 	(footprint "Capacitor_SMD:C_0805_2012Metric"
 		(layer "F.Cu")
-		(at 119.5 64.45 90)
+		(at 116.459 73.726 90)
 		(descr "Capacitor SMD 0805 (2012 Metric), square (rectangular) end terminal, IPC_7351 nominal, (Body size source: IPC-SM-782 page 76, https://www.pcb-3d.com/wordpress/wp-content/uploads/ipc-sm-782a_amendment_1_and_2.pdf, https://docs.google.com/spreadsheets/d/1BsfQQcO9C6DZCsRaXUlFlo91Tg2WpOkGARC1WS5S8t0/edit?usp=sharing), generated with kicad-footprint-generator")
 		(tags "capacitor")
@@
 	(footprint "Capacitor_SMD:C_0603_1608Metric"
 		(layer "F.Cu")
-		(at 118.28 72.22 90)
+		(at 118.28 73.66 90)
 		(descr "Capacitor SMD 0603 (1608 Metric), square (rectangular) end terminal, IPC_7351 nominal, (Body size source: IPC-SM-782 page 76, https://www.pcb-3d.com/wordpress/wp-content/uploads/ipc-sm-782a_amendment_1_and_2.pdf), generated with kicad-footprint-generator")
 		(tags "capacitor")

Commit message: Routing more
Parts:
- removed TP5, TP6: TestPoint, TestPoint:TestPoint_Loop_D2.60mm_Drill1.6mm_Beaded
- added TP_A1: TestPoint, TestPoint:TestPoint_Loop_D2.60mm_Drill1.6mm_Beaded, F.Cu at (89.0, 49.0)
- added TP_B1: TestPoint, TestPoint:TestPoint_Loop_D2.60mm_Drill1.6mm_Beaded, F.Cu at (89.0, 54.0)
- moved C5 9.59 mm to (120.7, 77.2)
- moved TP4 2.84 mm to (113.0, 65.0)
- moved R20 1.61 mm to (117.5, 89.2)
- moved Q11 1.61 mm to (115.1, 92.7)
- moved Q5 1.61 mm to (111.2, 91.7)
- moved Q6 1.61 mm to (115.0, 87.4)
- moved Q8 1.61 mm to (110.9, 86.4)
- moved R15 1.61 mm to (111.3, 94.3)
- moved R16 1.61 mm to (114.8, 84.9)
- moved R17 1.61 mm to (117.7, 95.4)
- moved R18 1.61 mm to (117.7, 92.4)
- moved R19 1.61 mm to (117.5, 86.1)
- moved R21 1.61 mm to (111.0, 88.9)
- moved R22 1.61 mm to (114.9, 90.5)
- moved R6 1.57 mm to (148.0, 88.4), turned to 90 degrees
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Routing:
- net +BATT: track 0.00 -> 78.3 mm
- net SOLAR_CURRENT_ADC: track 0.00 -> 35.6 mm, vias 0 -> 2
- net VSOLAR: track 0.00 -> 34.2 mm
- net /BuckBoost/VS_B: track 0.00 -> 18.2 mm
- net VDD: track 0.00 -> 15.8 mm
- net Net-(U3-Vs+): track 2.39 -> 17.2 mm
- net CELL_8V_ADC: track 0.00 -> 13.3 mm
- net /MCU/NRST: track 0.00 -> 9.93 mm, vias 0 -> 1
- net Net-(U4-LO): track 0.00 -> 8.84 mm
- net VSOLAR_ADC: track 0.00 -> 8.72 mm
- net Net-(U5-HO): track 0.00 -> 8.30 mm
- net GND: track 0.00 -> 7.73 mm
- net CELL_4V_ADC: track 0.00 -> 7.49 mm
- net /BuckBoost/VS_A: track 0.00 -> 7.36 mm
- net Net-(U4-HO): track 0.00 -> 7.19 mm
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Other:
- board size 68.2 x 38.2 mm -> 69 x 39 mm
