File: balance.kicad_sch (KiCad schematic)
At the start: 26 parts, among them Q10 AO3401A, Q11 2N7002, Q5 AO3401A, Q6 2N7002, Q7 2N7002, Q8 AO3401A

Commit message: Schematics updated P mosfets
Connections:
- net +BATT: now also Q5.2 (S); no longer Q5.3 (D)
- net CELL_4V: now also Q10.2 (S); no longer Q10.3 (D)
- net CELL_8V: now also Q8.2 (S); no longer Q8.3 (D)
- net at R26.1: now also Q10.3 (D); no longer Q10.2 (S)
- net at R22.1: now also Q8.3 (D); no longer Q8.2 (S)
- net at R16.1: now also Q5.3 (D); no longer Q5.2 (S)
Changed lines of the file:
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@@
 		(lib_id "Transistor_FET:AO3401A")
 		(at 93.98 52.07 0)
-		(unit 1)
-		(exclude_from_sim no)
-		(in_bom yes)
-		(on_board yes)
-		(dnp no)
-		(fields_autoplaced yes)
+		(mirror x)
+		(unit 1)
+		(exclude_from_sim no)
+		(in_bom yes)
+		(on_board yes)
+		(dnp no)
 		(property "Reference" "Q5"
-			(at 100.33 50.7999 0)
+			(at 100.33 53.3401 0)
 			(effects
 				(font
@@
 		)
 		(property "Value" "AO3401A"
-			(at 100.33 53.3399 0)
+			(at 100.33 50.8001 0)
 			(effects
 				(font
@@
 		)
 		(property "Footprint" "Package_TO_SOT_SMD:SOT-23"
-			(at 99.06 53.975 0)
+			(at 99.06 50.165 0)
 			(effects
 				(font
@@
 		)
 		(property "Datasheet" "http://www.aosmd.com/pdfs/datasheet/AO3401A.pdf"
-			(at 99.06 55.88 0)
+			(at 99.06 48.26 0)
 			(effects
 				(font
@@
 		(lib_id "Transistor_FET:AO3401A")
 		(at 166.37 52.07 0)
-		(unit 1)
-		(exclude_from_sim no)
-		(in_bom yes)
-		(on_board yes)
-		(dnp no)
-		(fields_autoplaced yes)
+		(mirror x)
+		(unit 1)
+		(exclude_from_sim no)
+		(in_bom yes)
+		(on_board yes)
+		(dnp no)
 		(property "Reference" "Q8"
-			(at 172.72 50.7999 0)
+			(at 172.72 53.3401 0)
 			(effects
 				(font
@@
 		)
 		(property "Value" "AO3401A"
-			(at 172.72 53.3399 0)
+			(at 172.72 50.8001 0)
 			(effects
 				(font
@@
 		)
 		(property "Footprint" "Package_TO_SOT_SMD:SOT-23"
-			(at 171.45 53.975 0)
+			(at 171.45 50.165 0)
 			(effects
 				(font
@@
 		)
 		(property "Datasheet" "http://www.aosmd.com/pdfs/datasheet/AO3401A.pdf"
-			(at 171.45 55.88 0)
+			(at 171.45 48.26 0)
 			(effects
 				(font
@@
 		(lib_id "Transistor_FET:AO3401A")
 		(at 241.3 52.07 0)
-		(unit 1)
-		(exclude_from_sim no)
-		(in_bom yes)
-		(on_board yes)
-		(dnp no)
-		(fields_autoplaced yes)
+		(mirror x)
+		(unit 1)
+		(exclude_from_sim no)
+		(in_bom yes)
+		(on_board yes)
+		(dnp no)
 		(property "Reference" "Q10"
-			(at 247.65 50.7999 0)
+			(at 247.65 53.3401 0)
 			(effects
 				(font
@@
 		)
 		(property "Value" "AO3401A"
-			(at 247.65 53.3399 0)
+			(at 247.65 50.8001 0)
 			(effects
 				(font
@@
 		)
 		(property "Footprint" "Package_TO_SOT_SMD:SOT-23"
-			(at 246.38 53.975 0)
+			(at 246.38 50.165 0)
 			(effects
 				(font
@@
 		)
 		(property "Datasheet" "http://www.aosmd.com/pdfs/datasheet/AO3401A.pdf"
-			(at 246.38 55.88 0)
-			(effects
-				(font
+			(at 246.38 48.26 0)
+			(effects
+				(font

Commit message: New design and layout
Parts:
- added R35, R36: 220k, Resistor_SMD:R_0402_1005Metric, symbol Device:R
- added R37, R38: 47.5k, Resistor_SMD:R_0402_1005Metric, symbol Device:R
- C18, C19: value 1n -> .1u; LCSC_Code C1588 -> C14663
- R27: value 390k -> 220k; footprint Resistor_SMD:R_0603_1608Metric -> Resistor_SMD:R_0402_1005Metric; LCSC_Code C23150 -> C851925; Tolerance (none) -> 0.5%
- R28: value 150k -> 220k; footprint Resistor_SMD:R_0603_1608Metric -> Resistor_SMD:R_0402_1005Metric; LCSC_Code C22807 -> C851925; Tolerance (none) -> 0.5%
- R29: value 150k -> 47.5k; footprint Resistor_SMD:R_0603_1608Metric -> Resistor_SMD:R_0402_1005Metric; LCSC_Code C22807 -> C319604; Tolerance (none) -> 0.5%
- R30: value 200k -> 47.5k; footprint Resistor_SMD:R_0603_1608Metric -> Resistor_SMD:R_0402_1005Metric; LCSC_Code C25811 -> C319604; Tolerance (none) -> 0.5%
Connections:
- net CELL_4V: now also R35.1, R36.1; no longer R29.1
- net CELL_4V_ADC: now also R35.2, R36.2, R37.2, R38.2; no longer R29.2, R30.2
- net CELL_8V: now also R28.1
- net CELL_8V_ADC: now also R29.2, R30.2
- net GND: now also R29.1, R37.1, R38.1; no longer R28.1

Commit message: Better balance resistors, fixes
Parts:
- R28: renamed from R16; footprint Resistor_SMD:R_0805_2012Metric -> Resistor_SMD:R_1206_3216Metric; LCSC_Code C17408 -> C17901
- R29: renamed from R22; footprint Resistor_SMD:R_0805_2012Metric -> Resistor_SMD:R_1206_3216Metric; LCSC_Code C17408 -> C17901
- R30: renamed from R26; footprint Resistor_SMD:R_0805_2012Metric -> Resistor_SMD:R_1206_3216Metric; LCSC_Code C17408 -> C17901
- renumbered C18 to C17, C19 to C18, Q7 to Q10, Q8 to Q6, Q10 to Q7, Q11 to Q8, Q6 to Q9, R15 to R19, R21 to R20, R25 to R21, R18 to R22, R19 to R23, R23 to R24, R17 to R25, R20 to R26, R24 to R27, R27 to R31, R28 to R32, R29 to R33, R30 to R34
