File: balance.kicad_sch (KiCad schematic)
At the start: 24 parts, among them Q10 AO3401A, Q11 2N7002, Q12 AO3401A, Q7 2N7002, Q8 AO3401A, Q9 2N7002

Commit message: Routing pt1
Parts:
- renumbered D13 to D11, D14 to D12, D15 to D13, Q11 to Q10, Q8 to Q5, Q10 to Q6, Q12 to Q7, Q7 to Q8, R27 to R19, R32 to R20, R37 to R21, R25 to R22, R30 to R23, R35 to R24, R26 to R25, R31 to R26, R36 to R27, R33 to R29, R38 to R30, R29 to R41, R34 to R42, R39 to R43
Changed lines of the file:
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@@
 		(dnp no)
 		(fields_autoplaced yes)
-		(property "Reference" "D14"
+		(property "Reference" "D12"
 			(at 184.15 65.0874 90)
 			(effects
@@
 			(project "JPBms2"
 				(path "/d86e471c-a8be-422d-a5d1-5a4699b7b766/220685a5-608c-4c12-9441-6825efcef07c"
-					(reference "D14")
+					(reference "D12")
 					(unit 1)
 				)
@@
 		(dnp no)
 		(fields_autoplaced yes)
-		(property "Reference" "#PWR048"
+		(property "Reference" "#PWR042"
 			(at 80.01 36.83 0)
 			(effects
@@
 			(project "JPBms2"
 				(path "/d86e471c-a8be-422d-a5d1-5a4699b7b766/220685a5-608c-4c12-9441-6825efcef07c"
-					(reference "#PWR048")
+					(reference "#PWR042")
 					(unit 1)
 				)
@@
 		(dnp no)
 		(fields_autoplaced yes)
-		(property "Reference" "R26"
+		(property "Reference" "R25"
 			(at 69.85 64.7699 0)
 			(effects
@@
 			(project "JPBms2"
 				(path "/d86e471c-a8be-422d-a5d1-5a4699b7b766/220685a5-608c-4c12-9441-6825efcef07c"
-					(reference "R26")
+					(reference "R25")
 					(unit 1)
 				)
@@
 		(dnp no)
 		(fields_autoplaced yes)
-		(property "Reference" "R36"
+		(property "Reference" "R27"
 			(at 217.17 64.7699 0)
 			(effects
@@
 			(project "JPBms2"
 				(path "/d86e471c-a8be-422d-a5d1-5a4699b7b766/220685a5-608c-4c12-9441-6825efcef07c"
-					(reference "R36")
+					(reference "R27")
 					(unit 1)
 				)
@@
 		(dnp no)
 		(fields_autoplaced yes)
-		(property "Reference" "R35"
+		(property "Reference" "R24"
 			(at 207.01 53.34 90)
 			(effects
@@
 			(project "JPBms2"
 				(path "/d86e471c-a8be-422d-a5d1-5a4699b7b766/220685a5-608c-4c12-9441-6825efcef07c"
-					(reference "R35")
+					(reference "R24")
 					(unit 1)
 				)
@@
 		(on_board yes)
 		(dnp no)
-		(property "Reference" "R34"
+		(property "Reference" "R42"
 			(at 178.054 76.2 90)
 			(effects
@@
 			(project "JPBms2"
 				(path "/d86e471c-a8be-422d-a5d1-5a4699b7b766/220685a5-608c-4c12-9441-6825efcef07c"
-					(reference "R34")
+					(reference "R42")
 					(unit 1)
 				)
@@
 		(on_board yes)
 		(dnp no)
-		(property "Reference" "R39"
+		(property "Reference" "R43"
 			(at 252.984 76.2 90)
 			(effects
@@
 			(project "JPBms2"
 				(path "/d86e471c-a8be-422d-a5d1-5a4699b7b766/220685a5-608c-4c12-9441-6825efcef07c"
-					(reference "R39")
+					(reference "R43")
 					(unit 1)
 				)
@@
 		(dnp no)
 		(fields_autoplaced yes)
-		(property "Reference" "Q7"
+		(property "Reference" "Q8"
 			(at 85.09 58.4199 0)
 			(effects
@@
 			(project "JPBms2"
 				(path "/d86e471c-a8be-422d-a5d1-5a4699b7b766/220685a5-608c-4c12-9441-6825efcef07c"
-					(reference "Q7")
+					(reference "Q8")
 					(unit 1)
 				)
@@
 		(dnp no)
 		(fields_autoplaced yes)
-		(property "Reference" "R31"
+		(property "Reference" "R26"
 			(at 142.24 64.7699 0)
 			(effects
@@
 			(project "JPBms2"
 				(path "/d86e471c-a8be-422d-a5d1-5a4699b7b766/220685a5-608c-4c12-9441-6825efcef07c"
-					(reference "R31")
+					(reference "R26")
 					(unit 1)
 				)
@@
 		(on_board yes)
 		(dnp no)
-		(property "Reference" "R29"
+		(property "Reference" "R41"
 			(at 105.664 76.2 90)
 			(effects
@@
 			(project "JPBms2"
 				(path "/d86e471c-a8be-422d-a5d1-5a4699b7b766/220685a5-608c-4c12-9441-6825efcef07c"
-					(reference "R29")
+					(reference "R41")
 					(unit 1)
 				)
@@
 		(dnp no)
 		(fields_autoplaced yes)
-		(property "Reference" "R32"
+		(property "Reference" "R20"
 			(at 156.21 43.1799 0)
 			(effects
@@
 			(project "JPBms2"
 				(path "/d86e471c-a8be-422d-a5d1-5a4699b7b766/220685a5-608c-4c12-9441-6825efcef07c"
-					(reference "R32")
+					(reference "R20")
 					(unit 1)
 				)
@@
 		(dnp no)
 		(fields_autoplaced yes)
-		(property "Reference" "#PWR051"
+		(property "Reference" "#PWR046"
 			(at 224.79 91.44 0)
 			(effects
@@
 			(project "JPBms2"
 				(path "/d86e471c-a8be-422d-a5d1-5a4699b7b766/220685a5-608c-4c12-9441-6825efcef07c"
-					(reference "#PWR051")
+					(reference "#PWR046")
 					(unit 1)
 				)
@@
 		(dnp no)
 		(fields_autoplaced yes)
-		(property "Reference" "Q11"
+		(property "Reference" "Q10"
 			(at 232.41 58.4199 0)
 			(effects
@@
 			(project "JPBms2"
 				(path "/d86e471c-a8be-422d-a5d1-5a4699b7b766/220685a5-608c-4c12-9441-6825efcef07c"
-					(reference "Q11")
+					(reference "Q10")
 					(unit 1)
 				)
@@
 		(dnp no)
 		(fields_autoplaced yes)
-		(property "Reference" "R38"
+		(property "Reference" "R30"
 			(at 246.38 68.5799 0)
 			(effects
@@
 			(project "JPBms2"
 				(path "/d86e471c-a8be-422d-a5d1-5a4699b7b766/220685a5-608c-4c12-9441-6825efcef07c"
-					(reference "R38")
+					(reference "R30")
 					(unit 1)
 				)
@@
 		(dnp no)
 		(fields_autoplaced yes)
-		(property "Reference" "#PWR052"
+		(property "Reference" "#PWR045"
 			(at 228.6 80.01 0)
 			(effects
@@
 			(project "JPBms2"
 				(path "/d86e471c-a8be-422d-a5d1-5a4699b7b766/220685a5-608c-4c12-9441-6825efcef07c"
-					(reference "#PWR052")
+					(reference "#PWR045")
 					(unit 1)
 				)
@@
 		(dnp no)
 		(fields_autoplaced yes)
-		(property "Reference" "R27"
+		(property "Reference" "R19"
 			(at 83.82 43.1799 0)
 			(effects
@@
 			(project "JPBms2"
 				(path "/d86e471c-a8be-422d-a5d1-5a4699b7b766/220685a5-608c-4c12-9441-6825efcef07c"
-					(reference "R27")
+					(reference "R19")
 					(unit 1)
 				)
@@
 		(dnp no)
 		(fields_autoplaced yes)
-		(property "Reference" "R30"
+		(property "Reference" "R23"
 			(at 132.08 53.34 90)
 			(effects
@@
 			(project "JPBms2"
 				(path "/d86e471c-a8be-422d-a5d1-5a4699b7b766/220685a5-608c-4c12-9441-6825efcef07c"
-					(reference "R30")
+					(reference "R23")
 					(unit 1)
 				)
@@
 		(dnp no)
 		(fields_autoplaced yes)
-		(property "Reference" "D13"
+		(property "Reference" "D11"
 			(at 111.76 65.0874 90)
 			(effects
@@
 			(project "JPBms2"
 				(path "/d86e471c-a8be-422d-a5d1-5a4699b7b766/220685a5-608c-4c12-9441-6825efcef07c"
-					(reference "D13")
+					(reference "D11")
 					(unit 1)
 				)
@@
 		(dnp no)
 		(fields_autoplaced yes)
-		(property "Reference" "R25"
+		(property "Reference" "R22"
 			(at 59.69 53.34 90)
 			(effects
@@
 			(project "JPBms2"
 				(path "/d86e471c-a8be-422d-a5d1-5a4699b7b766/220685a5-608c-4c12-9441-6825efcef07c"
-					(reference "R25")
+					(reference "R22")
 					(unit 1)
 				)
@@
 		(dnp no)
 		(fields_autoplaced yes)
-		(property "Reference" "R33"
+		(property "Reference" "R29"
 			(at 171.45 68.5799 0)
 			(effects
@@
 			(project "JPBms2"
 				(path "/d86e471c-a8be-422d-a5d1-5a4699b7b766/220685a5-608c-4c12-9441-6825efcef07c"
-					(reference "R33")
+					(reference "R29")
 					(unit 1)
 				)
@@
 		(on_board yes)
 		(dnp no)
-		(property "Reference" "Q8"
+		(property "Reference" "Q5"
 			(at 100.33 53.3401 0)
 			(effects
@@
 			(project "JPBms2"
 				(path "/d86e471c-a8be-422d-a5d1-5a4699b7b766/220685a5-608c-4c12-9441-6825efcef07c"
-					(reference "Q8")
+					(reference "Q5")
 					(unit 1)
 				)
@@
 		(on_board yes)
 		(dnp no)
-		(property "Reference" "Q10"
+		(property "Reference" "Q6"
 			(at 172.72 53.3401 0)
 			(effects
@@
 			(project "JPBms2"
 				(path "/d86e471c-a8be-422d-a5d1-5a4699b7b766/220685a5-608c-4c12-9441-6825efcef07c"
-					(reference "Q10")
+					(reference "Q6")
 					(unit 1)
 				)
@@
 		(dnp no)
 		(fields_autoplaced yes)
-		(property "Reference" "#PWR049"
+		(property "Reference" "#PWR043"
 			(at 81.28 80.01 0)
 			(effects
@@
 			(project "JPBms2"
 				(path "/d86e471c-a8be-422d-a5d1-5a4699b7b766/220685a5-608c-4c12-9441-6825efcef07c"
-					(reference "#PWR049")
+					(reference "#PWR043")
 					(unit 1)
 				)
@@
 		(on_board yes)
 		(dnp no)
-		(property "Reference" "Q12"
+		(property "Reference" "Q7"
 			(at 247.65 53.3401 0)
 			(effects
@@
 			(project "JPBms2"
 				(path "/d86e471c-a8be-422d-a5d1-5a4699b7b766/220685a5-608c-4c12-9441-6825efcef07c"
-					(reference "Q12")
+					(reference "Q7")
 					(unit 1)
 				)
@@
 		(dnp no)
 		(fields_autoplaced yes)
-		(property "Reference" "#PWR050"
+		(property "Reference" "#PWR044"
 			(at 153.67 80.01 0)
 			(effects
@@
 			(project "JPBms2"
 				(path "/d86e471c-a8be-422d-a5d1-5a4699b7b766/220685a5-608c-4c12-9441-6825efcef07c"
-					(reference "#PWR050")
+					(reference "#PWR044")
 					(unit 1)
 				)
@@
 		(dnp no)
 		(fields_autoplaced yes)
-		(property "Reference" "D15"
+		(property "Reference" "D13"
 			(at 259.08 65.0874 90)
 			(effects
@@
 			(project "JPBms2"
 				(path "/d86e471c-a8be-422d-a5d1-5a4699b7b766/220685a5-608c-4c12-9441-6825efcef07c"
-					(reference "D15")
+					(reference "D13")
 					(unit 1)
 				)
@@
 		(dnp no)
 		(fields_autoplaced yes)
-		(property "Reference" "R37"
+		(property "Reference" "R21"
 			(at 231.14 43.1799 0)
 			(effects
@@
 			(project "JPBms2"
 				(path "/d86e471c-a8be-422d-a5d1-5a4699b7b766/220685a5-608c-4c12-9441-6825efcef07c"
-					(reference "R37")
-					(unit 1)
-				)
+					(reference "R21")
+					(unit 1)
+				)
