File: adc.kicad_sch (KiCad schematic)
At the start: 28 parts, among them Q11 SK2301AW, Q12 SK2301AW, Q13 2N7002, Q14 SK2301AW, Q15 SK2301AW, Q16 2N7002, Q17 SK2301AW, Q18 SK2301AW, Q19 2N7002

Commit message: More accurate VBATT resistors, recalibrated vbatt off of vrefint, getting 0.5% accurate readings now
Parts:
- R6: LCSC_Code C23234 -> C728597
- R7: LCSC_Code C22847 -> C861205
Changed lines of the file:
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@@
 			)
 		)
-		(property "LCSC_Code" "C23234"
+		(property "LCSC_Code" "C728597"
 			(at 214.63 97.79 0)
 			(effects
@@
 			)
 		)
-		(property "LCSC_Code" "C22847"
-			(at 224.79 101.6 0)
-			(effects
+		(property "LCSC_Code" "C861205"
+			(at 224.79 101.6 0)
+			(effects
