File: buckboost.kicad_sch (KiCad schematic)
At the start: 29 parts, among them Q1 2N7002, Q2 AO3401A, Q3 AO3400A, Q4 AO3400A, Q5 AO3400A, Q6 AO3400A, U4 L6388E, U5 L6388E

Commit message: Routing pt1
Parts:
- renumbered C17 to C15, C18 to C20, D12 to D2, L1 to L2, Q3 to Q1, Q5 to Q2, Q1 to Q20, Q2 to Q21, Q4 to Q3, Q6 to Q4, R19 to R10, R20 to R11, R17 to R15, R18 to R16, R15 to R17, R16 to R18, R12 to R33, R13 to R34, R14 to R35, R23 to R36, R24 to R37, R22 to R8, R21 to R9, TP3 to TP5, TP4 to TP6, U5 to U6

Commit message: Starting cleanup
Parts:
- renumbered L2 to L1
Changed lines of the file:
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@@
 		(dnp no)
 		(fields_autoplaced yes)
-		(property "Reference" "L2"
+		(property "Reference" "L1"
 			(at 210.82 86.36 90)
 			(effects
@@
 			(project "JPBms2"
 				(path "/d86e471c-a8be-422d-a5d1-5a4699b7b766/0f5ad211-c4ad-40eb-a8ac-82970ee8fac9"
-					(reference "L2")
+					(reference "L1")
 					(unit 1)
 				)

Commit message: Board 1.3 ready -> fixed comparator inputs, balance LEDs, and TVS diode for battery disconnect protection
Parts:
- R36: value 7500 -> 56k; LCSC_Code C23234 -> C23206
- R37: value 1600 -> 4.7k; LCSC_Code C22847 -> C23162
Other:
- note added: "Vrefint = 1.224V We want the comparator to trigger when VS_A is just below the 16V TDS voltage. 15.8V * (4700/(56000+4700)) = 1.224"
- note removed: "Vrefint = 1.224V We want the comparator to trigger when VS_A is around 6V (or half the expected 12V) So we can have a backup measurement on when DCM mode is done"
Changed lines of the file:
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@@
 		)
 	)
-	(text "Vrefint = 1.224V\nWe want the comparator to trigger when VS_A is around 6V\n(or half the expected 12V)\nSo we can have a backup measurement on when DCM mode is done\n"
+	(text "Vrefint = 1.224V\nWe want the comparator to trigger when VS_A is \njust below the 16V TDS voltage.\n15.8V * (4700/(56000+4700)) = 1.224\n"
 		(exclude_from_sim no)
 		(at 248.158 142.494 0)
@@
 			)
 		)
-		(property "Value" "1600"
+		(property "Value" "4.7k"
 			(at 177.8 147.3199 0)
 			(effects
@@
 			)
 		)
-		(property "LCSC_Code" "C22847"
+		(property "LCSC_Code" "C23162"
 			(at 175.26 146.05 0)
 			(effects
@@
 			)
 		)
-		(property "Value" "7500"
+		(property "Value" "56k"
 			(at 177.8 137.1599 0)
 			(effects
@@
 			)
 		)
-		(property "LCSC_Code" "C23234"
+		(property "LCSC_Code" "C23206"
 			(at 175.26 135.89 0)
 			(effects
